File: GBC.kicad_sch (KiCad schematic)
At the start: 33 parts, among them J1 Conn_01x32_Female, J2 Conn_01x09_Male, U1 MAC-GBD, U2 M74VHC1GU04DFT1G-L22038, U3 FM28V100-TG, U4 3V0, U5 AM29F080B

Commit message: Add files via upload
Parts:
- removed LN1, LN2: L_Pack04, GBC:BLA2ABD121SN4D, symbol Device:L_Pack04
Connections:
- net D0 is gone; now on net DQ0: J1.22 (Pin_22), U1.32 (D0)
- net D1 is gone; now on net DQ1: J1.23 (Pin_23), U1.33 (D1)
- net D2 is gone; now on net DQ2: J1.24 (Pin_24), U1.34 (D2)
- net D3 is gone; now on net DQ3: J1.25 (Pin_25), U1.35 (D3)
- net D4 is gone; now on net DQ4: J1.26 (Pin_26), U1.36 (D4)
- net D5 is gone; now on net DQ5: J1.27 (Pin_27), U1.37 (D5)
- net D6 is gone; now on net DQ6: J1.28 (Pin_28), U1.39 (D6)
- net D7 is gone; now on net DQ7: J1.29 (Pin_29), U1.40 (D7)
Other:
- note added: "EMI Filter (deprecated)"
- note removed: "EMI Filter"
Changed lines of the file:
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@@
     (effects (font (size 1.27 1.27)) (justify left bottom))
   )
-  (text "EMI Filter" (at 170.18 52.07 0)
+  (text "EMI Filter\n(deprecated)" (at 170.18 54.61 0)
     (effects (font (size 1.27 1.27)) (justify left bottom))
   )
@@
     (effects (font (size 1.27 1.27)) (justify left bottom))
   )
-  (label "D2" (at 186.69 87.63 0)
-    (effects (font (size 1.27 1.27)) (justify left bottom))
-  )
   (label "RAM_A16" (at 222.25 76.2 180)
     (effects (font (size 1.27 1.27)) (justify right bottom))
@@
     (effects (font (size 1.27 1.27)) (justify left bottom))
   )
-  (label "D7" (at 106.68 120.65 270)
+  (label "DQ7" (at 106.68 120.65 270)
     (effects (font (size 1.27 1.27)) (justify right bottom))
   )
@@
     (effects (font (size 1.27 1.27)) (justify right bottom))
   )
-  (label "D5" (at 118.11 156.21 90)
+  (label "DQ5" (at 118.11 156.21 90)
     (effects (font (size 1.27 1.27)) (justify left bottom))
   )
@@
     (effects (font (size 1.27 1.27)) (justify right bottom))
   )
-  (label "DQ6" (at 176.53 69.85 180)
-    (effects (font (size 1.27 1.27)) (justify right bottom))
-  )
   (label "RAM_GND" (at 101.6 41.91 90)
     (effects (font (size 1.27 1.27)) (justify left bottom))
   )
-  (label "DQ1" (at 176.53 85.09 180)
-    (effects (font (size 1.27 1.27)) (justify right bottom))
-  )
   (label "3V0" (at 81.28 30.48 0)
     (effects (font (size 1.27 1.27)) (justify left bottom))
@@
     (effects (font (size 1.27 1.27)) (justify left bottom))
   )
-  (label "DQ2" (at 176.53 87.63 180)
-    (effects (font (size 1.27 1.27)) (justify right bottom))
-  )
   (label "ROM_A14" (at 232.41 123.19 180)
     (effects (font (size 1.27 1.27)) (justify right bottom))
@@
     (effects (font (size 1.27 1.27)) (justify left bottom))
   )
-  (label "D4" (at 96.52 120.65 270)
+  (label "DQ4" (at 96.52 120.65 270)
     (effects (font (size 1.27 1.27)) (justify right bottom))
   )
@@
     (effects (font (size 1.27 1.27)) (justify right bottom))
   )
-  (label "D4" (at 115.57 156.21 90)
+  (label "DQ4" (at 115.57 156.21 90)
     (effects (font (size 1.27 1.27)) (justify left bottom))
   )
@@
     (effects (font (size 1.27 1.27)) (justify left bottom))
   )
-  (label "D5" (at 186.69 67.31 0)
-    (effects (font (size 1.27 1.27)) (justify left bottom))
-  )
   (label "RAM_DQ6" (at 254 63.5 0)
     (effects (font (size 1.27 1.27)) (justify left bottom))
@@
     (effects (font (size 1.27 1.27)) (justify right bottom))
   )
-  (label "D6" (at 120.65 156.21 90)
+  (label "DQ6" (at 120.65 156.21 90)
     (effects (font (size 1.27 1.27)) (justify left bottom))
   )
@@
     (effects (font (size 1.27 1.27)) (justify left bottom))
   )
-  (label "D0" (at 105.41 156.21 90)
+  (label "DQ0" (at 105.41 156.21 90)
     (effects (font (size 1.27 1.27)) (justify left bottom))
   )
@@
     (effects (font (size 1.27 1.27)) (justify left bottom))
   )
-  (label "DQ0" (at 176.53 82.55 180)
-    (effects (font (size 1.27 1.27)) (justify right bottom))
-  )
   (label "RAM_A3" (at 254 91.44 0)
     (effects (font (size 1.27 1.27)) (justify left bottom))
@@
     (effects (font (size 1.27 1.27)) (justify left bottom))
   )
-  (label "D7" (at 123.19 156.21 90)
+  (label "DQ7" (at 123.19 156.21 90)
     (effects (font (size 1.27 1.27)) (justify left bottom))
   )
@@
     (effects (font (size 1.27 1.27)) (justify right bottom))
   )
-  (label "D6" (at 186.69 69.85 0)
-    (effects (font (size 1.27 1.27)) (justify left bottom))
-  )
   (label "A13" (at 232.41 125.73 180)
     (effects (font (size 1.27 1.27)) (justify right bottom))
@@
     (effects (font (size 1.27 1.27)) (justify left bottom))
   )
-  (label "D5" (at 99.06 120.65 270)
+  (label "DQ5" (at 99.06 120.65 270)
     (effects (font (size 1.27 1.27)) (justify right bottom))
   )
@@
     (effects (font (size 1.27 1.27)) (justify left bottom))
   )
-  (label "D0" (at 186.69 82.55 0)
-    (effects (font (size 1.27 1.27)) (justify left bottom))
-  )
-  (label "D4" (at 186.69 64.77 0)
-    (effects (font (size 1.27 1.27)) (justify left bottom))
-  )
   (label "A5" (at 77.47 156.21 90)
     (effects (font (size 1.27 1.27)) (justify left bottom))
@@
     (effects (font (size 1.27 1.27)) (justify left bottom))
   )
-  (label "D3" (at 186.69 90.17 0)
-    (effects (font (size 1.27 1.27)) (justify left bottom))
-  )
   (label "1V5" (at 71.12 41.91 90)
     (effects (font (size 1.27 1.27)) (justify left bottom))
@@
     (effects (font (size 1.27 1.27)) (justify right bottom))
   )
-  (label "D3" (at 113.03 156.21 90)
-    (effects (font (size 1.27 1.27)) (justify left bottom))
-  )
-  (label "D6" (at 104.14 120.65 270)
+  (label "DQ3" (at 113.03 156.21 90)
+    (effects (font (size 1.27 1.27)) (justify left bottom))
+  )
+  (label "DQ6" (at 104.14 120.65 270)
     (effects (font (size 1.27 1.27)) (justify right bottom))
   )
@@
     (effects (font (size 1.27 1.27)) (justify left bottom))
   )
-  (label "D2" (at 110.49 156.21 90)
+  (label "DQ2" (at 110.49 156.21 90)
     (effects (font (size 1.27 1.27)) (justify left bottom))
   )
@@
     (effects (font (size 1.27 1.27)) (justify left bottom))
   )
-  (label "D3" (at 93.98 120.65 270)
+  (label "DQ3" (at 93.98 120.65 270)
     (effects (font (size 1.27 1.27)) (justify right bottom))
   )
@@
     (effects (font (size 1.27 1.27)) (justify right bottom))
   )
-  (label "DQ3" (at 176.53 90.17 180)
-    (effects (font (size 1.27 1.27)) (justify right bottom))
-  )
   (label "3V0" (at 265.43 31.75 0)
     (effects (font (size 1.27 1.27)) (justify left bottom))
@@
     (effects (font (size 1.27 1.27)) (justify left bottom))
   )
-  (label "DQ7" (at 176.53 72.39 180)
-    (effects (font (size 1.27 1.27)) (justify right bottom))
-  )
   (label "5V0" (at 224.79 31.75 180)
     (effects (font (size 1.27 1.27)) (justify right bottom))
@@
     (effects (font (size 1.27 1.27)) (justify left bottom))
   )
-  (label "D1" (at 107.95 156.21 90)
+  (label "DQ1" (at 107.95 156.21 90)
     (effects (font (size 1.27 1.27)) (justify left bottom))
   )
@@
     (effects (font (size 1.27 1.27)) (justify left bottom))
   )
-  (label "DQ5" (at 176.53 67.31 180)
-    (effects (font (size 1.27 1.27)) (justify right bottom))
-  )
   (label "A10" (at 62.23 109.22 180)
     (effects (font (size 1.27 1.27)) (justify right bottom))
@@
     (effects (font (size 1.27 1.27)) (justify left bottom))
   )
-  (label "D7" (at 186.69 72.39 0)
-    (effects (font (size 1.27 1.27)) (justify left bottom))
-  )
   (label "GND" (at 132.08 120.65 270)
     (effects (font (size 1.27 1.27)) (justify right bottom))
@@
     (effects (font (size 1.27 1.27)) (justify left bottom))
   )
-  (label "DQ4" (at 176.53 64.77 180)
-    (effects (font (size 1.27 1.27)) (justify right bottom))
-  )
-  (label "D1" (at 186.69 85.09 0)
-    (effects (font (size 1.27 1.27)) (justify left bottom))
-  )
   (label "RAM_A1" (at 254 86.36 0)
     (effects (font (size 1.27 1.27)) (justify left bottom))
@@
     (effects (font (size 1.27 1.27)) (justify left bottom))
   )
-  (label "D1" (at 88.9 120.65 270)
+  (label "DQ1" (at 88.9 120.65 270)
     (effects (font (size 1.27 1.27)) (justify right bottom))
   )
@@
     (effects (font (size 1.27 1.27)) (justify right bottom))
   )
-  (label "D2" (at 91.44 120.65 270)
-    (effects (font (size 1.27 1.27)) (justify right bottom))
-  )
-  (label "D0" (at 86.36 120.65 270)
+  (label "DQ2" (at 91.44 120.65 270)
+    (effects (font (size 1.27 1.27)) (justify right bottom))
+  )
+  (label "DQ0" (at 86.36 120.65 270)
     (effects (font (size 1.27 1.27)) (justify right bottom))
   )
@@
     (pin "1")
     (pin "2")
-  )
-  (symbol (lib_id "Device:L_Pack04") (at 181.61 69.85 270) (unit 1)
-    (in_bom yes) (on_board yes) (fields_autoplaced)
-    (property "Reference" "LN1" (id 0) (at 181.61 58.42 90))
-    (property "Value" "L_Pack04" (id 1) (at 181.61 60.96 90))
-    (property "Footprint" "GBC:BLA2ABD121SN4D" (id 2) (at 184.15 76.2 90)
-      (effects (font (size 1.27 1.27)) hide)
-    )
-    (property "Datasheet" "~" (id 3) (at 184.15 76.2 90)
-      (effects (font (size 1.27 1.27)) hide)
-    )
-    (pin "1")
-    (pin "2")
-    (pin "3")
-    (pin "4")
-    (pin "5")
-    (pin "6")
-    (pin "7")
-    (pin "8")
   )
   (symbol (lib_id "Connector:Conn_01x32_Female") (at 90.17 161.29 90) (mirror x) (unit 1)
@@
     (pin "5")
   )
-  (symbol (lib_id "Device:L_Pack04") (at 181.61 87.63 270) (unit 1)
-    (in_bom yes) (on_board yes) (fields_autoplaced)
-    (property "Reference" "LN2" (id 0) (at 181.61 76.2 90))
-    (property "Value" "L_Pack04" (id 1) (at 181.61 78.74 90))
-    (property "Footprint" "GBC:BLA2ABD121SN4D" (id 2) (at 184.15 93.98 90)
-      (effects (font (size 1.27 1.27)) hide)
-    )
-    (property "Datasheet" "~" (id 3) (at 184.15 93.98 90)
-      (effects (font (size 1.27 1.27)) hide)
-    )
-    (pin "1")
-    (pin "2")
-    (pin "3")
-    (pin "4")
-    (pin "5")
-    (pin "6")
-    (pin "7")
-    (pin "8")
-  )
   (symbol (lib_id "Device:C") (at 270.51 157.48 0) (unit 1)
     (in_bom yes) (on_board yes) (fields_autoplaced)
@@
       (reference "J2") (unit 1) (value "Conn_01x09_Male") (footprint "GBC:JST_B9B-ZR-SM4-Flat")
     )
-    (path "/210522d3-5635-4329-b7af-ace86f31e626"
-      (reference "LN1") (unit 1) (value "L_Pack04") (footprint "GBC:BLA2ABD121SN4D")
-    )
-    (path "/f14dfab8-99e0-4c25-9707-21081698485f"
-      (reference "LN2") (unit 1) (value "L_Pack04") (footprint "GBC:BLA2ABD121SN4D")
-    )
     (path "/fccaeff6-49ba-45ca-b8f7-900d9130b2fd"

Commit message: Add files via upload
Parts:
- removed C16: 22p, Capacitor_SMD:C_0603_1608Metric, symbol Device:C
- renumbered C20 to C1, C9 to C10, C10 to C12, C19 to C13, C12 to C14, C13 to C15, C14 to C16, C15 to C17, C17 to C18, C18 to C19, C1 to C2, C2 to C3, C3 to C4, C4 to C5, C5 to C6, C6 to C7, C7 to C8, C8 to C9

Commit message: Add files via upload
Parts:
- C10: value 22p -> 39p
Other:
- company: (none) -> Made by 2BitWizard
- title: (none) -> Flashable Camera
